Commit message: gazebo simulation added

File: src/robotic_arm_desc/urdf/robotic_arm.urdf (robot description, URDF)
Before this commit: robot roboticarm_desc, 8 links, 7 joints
Links:
- link base_link: geometry collision box size=0.05 0.05 0.05; visual mesh filename=package://robotic_arm_desc/meshes/base_link.STL
- link link_1: geometry collision mesh filename=package://robotic_arm_desc/meshes/link_1.STL; visual mesh filename=package://robotic_arm_desc/meshes/link_1.STL
- link link_2: geometry collision mesh filename=package://robotic_arm_desc/meshes/link_2.STL; visual mesh filename=package://robotic_arm_desc/meshes/link_2.STL
- link link_3: geometry collision mesh filename=package://robotic_arm_desc/meshes/link_3.STL; visual mesh filename=package://robotic_arm_desc/meshes/link_3.STL
- link link_4: geometry collision mesh filename=package://robotic_arm_desc/meshes/link_4.STL; visual mesh filename=package://robotic_arm_desc/meshes/link_4.STL
- link link_5: geometry collision mesh filename=package://robotic_arm_desc/meshes/link_5.STL; visual mesh filename=package://robotic_arm_desc/meshes/link_5.STL
- link link_6: geometry collision mesh filename=package://robotic_arm_desc/meshes/link_6.STL; visual mesh filename=package://robotic_arm_desc/meshes/link_6.STL
