Commit message: gazebo and moveit added successfully

File: src/robotic_arm_desc/urdf/robotic_arm.urdf.xacro (robot description, xacro)
@@ -4,5 +4,16 @@
      For more information, please see http://wiki.ros.org/sw_urdf_exporter -->
 <robot
-  name="robotic_arm_desc">
+  name="robotic_arm_desc"
+   xmlns:xacro="http://www.ros.org/wiki/xacro"
+  >
+  <xacro:arg name="use_gazebo" default="false"/>
+  <xacro:property name="mesh_pkg" value="package://robotic_arm_desc/meshes"/>
+  <xacro:if value="$(arg use_gazebo)">
+    <xacro:include filename="$(find robotic_arm_desc)/urdf/gazebo_ros2_control.xacro"/>
+    <xacro:include filename="$(find robotic_arm_desc)/urdf/gazebo.xacro"/>
+  </xacro:if>
+  <xacro:unless value="$(arg use_gazebo)">
+    <xacro:include filename="$(find robotic_arm_desc)/urdf/ros2_control.xacro"/>
+  </xacro:unless>
   <link
     name="base_link">
@@ -26,6 +37,5 @@
         rpy="0 0 0" />
       <geometry>
-        <mesh
-          filename="package://robotic_arm_desc/meshes/base_link.STL" />
+        <mesh filename="${mesh_pkg}/base_link.STL"/>
       </geometry>
       <material
@@ -35,13 +45,12 @@
       </material>
     </visual>
-    <!-- <collision>
-      <origin
-        xyz="0 0 0"
-        rpy="0 0 0" />
-      <geometry>
-        <mesh
-          filename="package://robotic_arm_desc/meshes/base_link.STL" />
-      </geometry>
-    </collision> -->
+    <collision>
+      <origin
+        xyz="0 0 0"
+        rpy="0 0 0" />
+      <geometry>
+        <mesh filename="${mesh_pkg}/base_link.STL"/>
+      </geometry>
+    </collision>
     <collision>
       <geometry>
@@ -71,6 +80,5 @@
         rpy="0 0 0" />
       <geometry>
-        <mesh
-          filename="package://robotic_arm_desc/meshes/link_1.STL" />
+        <mesh filename="${mesh_pkg}/link_1.STL"/>
       </geometry>
       <material
@@ -85,6 +93,5 @@
         rpy="0 0 0" />
       <geometry>
-        <mesh
-          filename="package://robotic_arm_desc/meshes/link_1.STL" />
+        <mesh filename="${mesh_pkg}/link_1.STL"/>
       </geometry>
     </collision>
@@ -129,6 +136,5 @@
         rpy="0 0 0" />
       <geometry>
-        <mesh
-          filename="package://robotic_arm_desc/meshes/link_2.STL" />
+        <mesh filename="${mesh_pkg}/link_2.STL"/>
       </geometry>
       <material
@@ -143,6 +149,5 @@
         rpy="0 0 0" />
       <geometry>
-        <mesh
-          filename="package://robotic_arm_desc/meshes/link_2.STL" />
+        <mesh filename="${mesh_pkg}/link_2.STL"/>
       </geometry>
     </collision>
@@ -187,6 +192,5 @@
         rpy="0 0 0" />
       <geometry>
-        <mesh
-          filename="package://robotic_arm_desc/meshes/link_3.STL" />
+        <mesh filename="${mesh_pkg}/link_3.STL"/>
       </geometry>
       <material
@@ -201,6 +205,5 @@
         rpy="0 0 0" />
       <geometry>
-        <mesh
-          filename="package://robotic_arm_desc/meshes/link_3.STL" />
+        <mesh filename="${mesh_pkg}/link_3.STL"/>
       </geometry>
     </collision>
@@ -245,6 +248,5 @@
         rpy="0 0 0" />
       <geometry>
-        <mesh
-          filename="package://robotic_arm_desc/meshes/link_4.STL" />
+        <mesh filename="${mesh_pkg}/link_4.STL"/>
       </geometry>
       <material
@@ -259,6 +261,5 @@
         rpy="0 0 0" />
       <geometry>
-        <mesh
-          filename="package://robotic_arm_desc/meshes/link_4.STL" />
+        <mesh filename="${mesh_pkg}/link_4.STL"/>
       </geometry>
     </collision>
@@ -301,6 +302,5 @@
       <origin xyz="0 0 -0.04" rpy="0 0 0"/>
       <geometry>
-        <mesh
-          filename="package://robotic_arm_desc/meshes/link_5.STL" />
+        <mesh filename="${mesh_pkg}/link_5.STL"/>
       </geometry>
       <material
@@ -313,6 +313,5 @@
       <origin xyz="0 0 -0.04" rpy="0 0 0"/>
       <geometry>
-        <mesh
-          filename="package://robotic_arm_desc/meshes/link_5.STL" />
+        <mesh filename="${mesh_pkg}/link_5.STL"/>
       </geometry>
     </collision>
@@ -340,5 +339,5 @@
       <origin xyz="0 0 -0.04" rpy="0 0 0"/>
       <geometry>
-        <mesh filename="package://robotic_arm_desc/meshes/link_6.STL"/>
+        <mesh filename="${mesh_pkg}/link_6.STL"/>
       </geometry>
       <material name="">
@@ -349,5 +348,5 @@
       <origin xyz="0 0 -0.04" rpy="0 0 0"/>
       <geometry>
-        <mesh filename="package://robotic_arm_desc/meshes/link_6.STL"/>
+        <mesh filename="${mesh_pkg}/link_6.STL"/>
       </geometry>
     </collision>
@@ -366,40 +365,11 @@
     <origin xyz="0 0 0.09" rpy="0 0 0"/>
   </joint>
-  <ros2_control name="MyRobotSystem" type="system">
-  <hardware>
-    <plugin>gz_ros2_control/GazeboSimSystem</plugin>
-  </hardware>
-  <joint name="joint_1">
-    <command_interface name="position"/>
-    <state_interface name="position"/>
-  </joint>
-  <joint name="joint_2">
-    <command_interface name="position"/>
-    <state_interface name="position"/>
-  </joint>
-  <joint name="joint_3">
-    <command_interface name="position"/>
-    <state_interface name="position"/>
-  </joint>
-  <joint name="joint_4">
-    <command_interface name="position"/>
-    <state_interface name="position"/>
-  </joint>
-  <joint name="joint_5">
-    <command_interface name="position"/>
-    <state_interface name="position"/>
-  </joint>
-  <joint name="joint_6">
-    <command_interface name="position"/>
-    <state_interface name="position"/>
-  </joint>
-  </ros2_control>
-  <gazebo>
-  <plugin filename="libgz_ros2_control-system.so"
-          name="gz_ros2_control::GazeboSimROS2ControlPlugin">
-    <parameters>
-      /home/rounak/projects/robotic_arm_4dof_ws/install/robotic_arm_desc/share/robotic_arm_desc/config/controllers.yaml
-    </parameters>
-  </plugin>
-</gazebo>
+  <xacro:if value="$(arg use_gazebo)">
+    <xacro:robotic_arm_desc_ros2_control
+        name="MyRobotSystem"/>
+  </xacro:if>
+  <xacro:unless value="$(arg use_gazebo)">
+    <xacro:robotic_arm_desc_ros2_control
+        name="MyRobotSystem"/>
+  </xacro:unless>
 </robot>

File: src/robotic_arm_moveit_config/config/robotic_arm_desc.ros2_control.xacro (robot description, xacro)
@@ -1,5 +1,5 @@
 <?xml version="1.0"?>
 <robot xmlns:xacro="http://www.ros.org/wiki/xacro">
-    <xacro:macro name="roboticarm_desc_ros2_control" params="name initial_positions_file">
+    <xacro:macro name="robotic_arm_desc_ros2_control" params="name initial_positions_file">
         <xacro:property name="initial_positions" value="${xacro.load_yaml(initial_positions_file)['initial_positions']}"/>
         <ros2_control name="${name}" type="system">
